File: Assignments/1.Pragadish Selvan R/Assignment-1/Home Automation/Brave Densor.brd (EAGLE design)
At the start: 89.4 x 92 mm, 4 parts, among them U1 ARDUINO-UNO-R3-SHIELD

Commit message: Sept 25
Parts:
- removed D1: RED, Tinkercad:LEDRD254W60D565H860B
- added GAS1: GAS-SENSORMQ-XX-SOCKET, Tinkercad:MQ-XX-SOCKET
- added K1, K2: RELAY-SPDT_LU-5-R, Tinkercad:LU-5-R
- added L1, L2: LIGHTBULB, Tinkercad:1X02
- added M1: MOTOR_HDR, Tinkercad:MOTOR
- added P1: BATTERYGENERIC, Tinkercad:BATTERY-GENERIC
- added PIEZO1: PIEZO, Tinkercad:PIEZO
- added PIR1: PIR-SENSOR_28027, Tinkercad:28027
- added R1: PHOTOCELL_GL5528, Tinkercad:GL5528
- added R3: 5k, Tinkercad:RESAD1016W63L850D250B
- added S1: TOGGLE, Tinkercad:SWITCH-SPDT-PTH-8.5X3.7MM
- added SERVO1: SERVOSG90, Tinkercad:SG90
- moved R2 111.9 mm to (130.6, 60.6), turned to 90 degrees
- moved PING1 92.9 mm to (138.0, 26.4), turned to 180 degrees
- moved U1 19.3 mm to (29.8, 36.6), turned to 180 degrees
Connections:
- removed net D1_A: D1.1, R2.1
- removed net U1_D3: PING1.3, U1.D3
- new net L2_1: K2.12, L2.1
- new net L2_2: L1.2, L2.2
- new net M1_+: M1.+, S1.1
- new net M1_-: K1.6, M1.-
- new net P1+: K2.6, P1.+, S1.2
- new net P1-: K1.12, L1.1, P1.-
- new net U1_A0: R1.1, R2.2, U1.A0
- new net U1_A1: GAS1.1, GAS1.3, R3.1, U1.A1
- new net U1_D10: K1.8, U1.D10
- new net U1_D13: K2.5, U1.D13
- new net U1_D6: PING1.3, U1.D6
- new net U1_D7: SERVO1.3, U1.D7
- new net U1_D8: PIEZO1.1, U1.D8
- net U1_5V: now also GAS1.4, GAS1.5, GAS1.6, PIR1.2, R2.1, SERVO1.2
- net U1_D9: now also PIR1.1; no longer R2.2
- net U1_GND: now also GAS1.2, K1.5, K2.8, PIEZO1.2, PIR1.3, R1.2, R3.2, SERVO1.1; no longer D1.2
Other:
- board size 89.4 x 92 mm -> 373 x 126.2 mm
